File: motors_and_encoders.kicad_sch (KiCad schematic)
At the start: 18 parts, among them J10 Conn_01x02, J11 Conn_01x02, J13 Conn_01x02, J2 Conn_01x06, J3 Conn_01x06, U1 ROB-14450, U5 74HC14, U6 74LVC2G14

Commit message: Update readme
Changed lines of the file:
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@@
 					(size 1.27 1.27)
 				)
+				(hide yes)
 			)
 		)
@@
 					(size 1.27 1.27)
 				)
+				(hide yes)
 			)
 		)
@@
 					(size 1.27 1.27)
 				)
+				(hide yes)
 			)
 		)
@@
 					(size 1.27 1.27)
 				)
+				(hide yes)
 			)
 		)
@@
 					(size 1.27 1.27)
 				)
-			)
-		)
+				(hide yes)
+			)
+		)
